File: hardware/MAXwell.kicad_pcb (KiCad board)
At the start: 2 copper layers, 85.9 x 96.1 mm, 155 parts, among them J1 Conn_02x05_Odd_Even, J2 Conn_02x12_Counter_Clockwise, J3 Barrel_Jack_Switch_Pin3Ring, SW1 SW_Push_Dual, SW10 SW_Wuerth_450301014042, SW11 SW_Wuerth_450301014042, SW12 SW_Wuerth_450301014042, SW13 SW_Wuerth_450301014042, SW2 SW_Push_Dual, SW3 SW_Push_Dual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

Commit message: established ground planes
Routing:
- net +3V3: track 429.8 -> 616.3 mm, vias 22 -> 42
- net Net-(U5-IO1_4): track 71.7 -> 67.5 mm
- net Net-(U5-IO1_21): track 33.7 -> 31.1 mm
- net Net-(U5-IO1_19): track 63.7 -> 61.1 mm
- net Net-(U5-IO1_12/GCLK0): track 22.7 -> 20.7 mm
- net Net-(U5-IO1_29): track 55.9 -> 54.0 mm
- net Net-(J1-Pin_5): track 74.6 -> 72.8 mm, vias 8 -> 6
- net Net-(U5-IO1_8): track 65.1 -> 63.5 mm
- net Net-(U5-IO2_55): track 44.6 -> 43.1 mm
- net GND: track 170.2 -> 168.8 mm, vias 52 -> 167
- net Net-(U5-IO2_61): track 57.8 -> 56.4 mm
- net Net-(U5-IO2_95): track 22.8 -> 23.9 mm
- net Net-(U5-IO1_3): track 73.8 -> 72.8 mm
- net Net-(U5-IO2_58): track 38.6 -> 39.6 mm
- net Net-(U5-IO1_20): track 45.9 -> 44.9 mm
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- added copper zone on F.Cu, net GND
Other:
- board text added: "MAXwell FPGA Board Michael Hohenstein"
